File: P1001-001 - 16bit CPU/P1001-001-003-320 - Controller/P1001-001-003-320 - Controller.brd (EAGLE design)
At the start: 200 x 48 mm, 80 parts, among them IC1 74LS138D, IC14 74LS138D, IC3 74LS138D, IC4 74LS138D, IC5 74LS138D, J1 22-27-2041-04

Commit message: Added the simple reg, cleaned things up
Parts:
- removed ADD6, A_SWAP1, A_SWAP2, XOR7: (no value), led:SFH482
- removed JP1, JP2, JP20: (no value), jumper:JP1
- removed JP10, JP15, JP4, JP6, JP7: (no value), jumper:JP4
- removed JP14: (no value), jumper:JP2W
- added ALU_HIGH, ALU_LOW, A_IN_LOW, A_OUT2, B_IN_LOW, B_OUT2, RAN_IN_2: (no value), jumper:JP4
- added A_IN_HIGH, B_IN_HIGH, RAM_PC_OUT, RAN_IN_3: (no value), jumper:JP1
- added PC_OUT, RAM_OUT: (no value), led:SFH482
- added RAN_IN_1: (no value), jumper:JP2W
- added SV1: (no value), con-harting-ml:ML16
- moved PC_INC 130.0 mm to (174.0, 27.0)
- moved C_INC 128.3 mm to (53.0, 27.0)
- moved NEXT_INS 119.5 mm to (136.0, 27.0)
- moved C_OUT 119.3 mm to (65.0, 27.0)
- moved IC3 118.9 mm to (169.0, 40.0), flipped to the bottom, turned to 90 degrees
- moved HALT 116.7 mm to (142.0, 27.0)
- moved RESET 113.9 mm to (148.0, 27.0)
- moved C_IN 112.2 mm to (47.0, 27.0)
- moved D_REG 107.0 mm to (58.0, 37.0)
- moved D_OUT 106.9 mm to (84.0, 27.0)
- moved C_REG 105.5 mm to (63.0, 44.0)
- moved C_DEC 101.1 mm to (59.0, 27.0)
- moved PC_IN 99.0 mm to (168.0, 27.0)
- moved D_IN 97.1 mm to (72.0, 27.0)
- moved RAM_IN_H 96.7 mm to (143.0, 18.0)
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Connections:
- removed net N$37: IC14.9, XOR7.K
- removed net N$42: R5.15, XOR7.A
- removed net N$43: B_IN_H_L.A, R4.15
- removed net N$50: B_IN_H_L.K, IC1.9
- new net IR10: SV1.11
- new net IR11: SV1.12
- new net IR12: SV1.13
- new net IR13: SV1.14
- new net IR14: SV1.15
- new net IR15: SV1.16
- new net IR8: SV1.9
- new net IR9: SV1.10
- net A-CLEAR: now also A_IN_LOW.4; no longer JP15.4
- net ADD: now also ALU_LOW.1; no longer JP10.1
- net AND: now also ALU_HIGH.3; no longer JP4.3
- net A_HIGH: now also A_OUT2.2
- net A_IN: now also A_IN_LOW.3; no longer JP15.3
- net A_IN_H_H: now also A_IN_LOW.1; no longer JP15.1
- net A_IN_H_L: now also A_IN_HIGH.1; no longer JP20.1
- net A_IN_L_H: now also A_IN_HIGH.2; no longer JP20.2
- net A_IN_L_L: now also A_IN_LOW.2; no longer JP15.2
- net A_LOW: now also A_OUT2.3
- net A_OUT: now also A_OUT2.4
- net A_SWAP: now also A_OUT2.1
- net BUS13: now also RAN_IN_3.2; no longer JP2.2
- net BUS14: now also RAN_IN_3.1; no longer JP2.1
- net BUS15: now also RAN_IN_2.4; no longer JP7.4
- net BUS16: now also RAN_IN_2.3; no longer JP7.3
- net BUS17: now also RAN_IN_2.2; no longer JP7.2
- net BUS21: now also RAN_IN_2.1; no longer JP7.1
- net BUS26: now also RAN_IN_1.3; no longer JP14.3
- net BUS27: now also RAN_IN_1.2; no longer JP14.2
- net BUS28: now also RAN_IN_1.1; no longer JP14.1
- net B_CLEAR: now also B_IN_LOW.4; no longer JP6.4
- net B_HIGH: now also B_OUT2.2
- net B_IN: now also B_IN_LOW.3; no longer JP6.3
- net B_IN_H_H: now also B_IN_LOW.1; no longer JP6.1
- net B_IN_H_L: now also B_IN_HIGH.1, B_IN_H_L.K; no longer ADD6.K, JP1.1
- net B_IN_L_H: now also B_IN_HIGH.2; no longer JP1.2
- net B_IN_L_L: now also B_IN_LOW.2; no longer JP6.2
- net B_LOW: now also B_OUT2.3
- net B_OUT: now also B_OUT2.4
- net B_SWAP: now also B_OUT2.1
- net N$36: now also B_IN_H_L.A; no longer ADD6.A
- net N$44: now also RAM_OUT.A, RAM_PC_OUT.2; no longer A_SWAP1.A
- net N$54: now also PC_OUT.A, RAM_PC_OUT.1; no longer A_SWAP2.A
- net NOT: now also ALU_HIGH.1; no longer JP4.1
- net OR: now also ALU_HIGH.2; no longer JP4.2
- net PC_OUT: now also PC_OUT.K; no longer A_SWAP2.K
- net RAM_OUT: now also RAM_OUT.K; no longer A_SWAP1.K
- net SHL: now also ALU_LOW.3; no longer JP10.3
- net SHR: now also ALU_LOW.4; no longer JP10.4
- net SUB: now also ALU_LOW.2; no longer JP10.2
- net XOR: now also ALU_HIGH.4; no longer JP4.4
