File: P1001-001 - 16bit CPU/P1001-001-003-320 - Controller/P1001-001-003-320 - Controller.sch (EAGLE design)
At the start: 108 parts, among them IC1 74LS138D, IC10 74ALS00D, IC11 74ABT164D, IC12 74ABT164D, IC13 74ABT164D, IC14 74LS138D, IC15 74ABT164D, IC16 74ABT164D, IC17 74ABT164D, IC18 74ABT164D, IC19 74ABT164D, IC2 74LS157D, IC20 74ABT164D, IC3 74LS138D, IC4 74LS138D, IC5 74LS138D, IC6 74LS157D, IC7 74LS157D, IC8 74LS157D, IC9 74LS157D, J1 22-27-2041-04

Commit message: Add the control board
Parts:
- removed ALU_HIGH, ALU_LOW, A_OUT2, B_IN_LOW, B_OUT2, C_REG, RAN_IN_2, STACK: (no value), jumper:JP4E
- removed A_CLEAR, B_CLEAR, D_IN, RAM_IN_LOW, X_SWAP: (no value), led:LEDSFH482
- removed BACKBUS, FRONTBUS: (no value), con-harting-ml:ML16
- removed B_IN_HIGH, RAM_PC_OUT, RAN_IN_3: (no value), jumper:JP1E
- removed D_REG, RAN_IN_1, X_REG: (no value), jumper:JP2W
- removed IC14: 74LS138D, 74xx-us:74LS138D
- added ABC_CLEAR, B_IN_LOW1, HALT_RESEDT_NEXTINS, PC_MAR_IR_IN, RAM_STACK_IN: (no value), jumper:JP2W
- added ADD_SUB, B_IN_HIGH1, CLEAR_OUNS, EXTRA_1_2_PINS, EXTRA_3_4_PINS, EXTRA_5_6_PINS, INTERUPTS, PC_INC_DEC, RAM_IMT_OUT: (no value), jumper:JP1E
- added A_CLEAR_LED, B_CLEAR_LED, D_CLEAR_LED, D_HIGH, D_IN_H, D_IN_L, D_LOW, EXTRA1, EXTRA2, EXTRA3, EXTRA4, EXTRA5, EXTRA6, EXTRA_OUT1, EXTRA_OUT2, EXTRA_OUT3, EXTRA_OUT4, INTERUPT_OUT, PAUSE_INERUPT, PC_DEC, PLAY_INTERUPT, RAM_IN_L, ROL, ROR, STEP1, STEP2, STEP3, STEP4: (no value), led:LEDSFH482
- added A_OUT_PINS, B_OUT_PIMS, C_X_OC_STACK_OUT, D_OUT_PINS, EXTRA_OUT, IN_C_D_X, LOGIC_OP, SHIFT_ROLL, STACK_C, STEP_PINS: (no value), jumper:JP4E
- added BANKA: SST39VF1602-70-4I-EKE, 16bit:SST39VF1602-70-4I-EKE
- added IC21, IC22, IC23: 74LS138D, 74xx-us:74LS138D
- added IC27: MEGA8535-A, atmel:MEGA8535-A
- added PULL_DOWN, R12, R13, R14: (no value), rcl:R-US_M0805
- added R10, R7, R8: (no value), resistor-bourns:2NBS16-15
- added READ_WRITE: (no value), jumper:JP2E
- added RN2: (no value), resistor-dil:10R-NSOMC
- added SV3: (no value), con-harting-ml:ML16
- added SV5: (no value), con-harting-ml:ML6
- A_IN_LOW: device jumper:JP4E -> jumper:JP2W
- JP4: device jumper:JP1E -> jumper:JP3Q
- U$1: value SST39VF1602-70-4I-EKE -> 4-DIGIT-7-SEGMENT; device 16bit:SST39VF1602-70-4I-EKE -> ADAFRUIT:4-DIGIT-7-SEGMENT
- renumbered IC11 to ADD_LOW, IC12 to ADD_MID, IC13 to ADD_HIGH, IC15 to BA_LOW, IC16 to BA_HIGH, IC17 to BB_LOW, IC18 to BB_HIGH, IC19 to BC_LOW, IC2 to SW_PROD_3, IC20 to BC_HIGH, IC6 to SW_PROD_2, IC7 to SW_PROD_1, IC8 to SW_PROD_4, IC9 to SW_PROD_5, JP5 to POWER_PINS, U$2 to BANKB, U$3 to BANKC
Connections:
- removed net A-CLEAR: A_CLEAR.C, A_IN_LOW.4, IC14A.Y0
- removed net ADD: ADD.C, ALU_LOW.1, IC3A.Y0
- removed net AND: ALU_HIGH.3, AND.C, IC3A.Y6
- removed net A_HIGH: A_HIGH.C, A_OUT2.2, IC5A.Y1
- removed net A_IN: A_IN.C, A_IN_LOW.3, IC14A.Y1
- removed net A_IN_H_H: A_IN_H_H.C, A_IN_LOW.1, IC14A.Y3
- removed net A_IN_H_L: A_IN_HIGH.1, A_IN_H_L.C, IC14A.Y5
- removed net A_IN_L_H: A_IN_HIGH.2, A_IN_L_H.C, IC14A.Y4
- removed net A_IN_L_L: A_IN_LOW.2, A_IN_L_L.C, IC14A.Y2
- removed net A_LOW: A_LOW.C, A_OUT2.3, IC5A.Y2
- removed net A_OUT: A_OUT.C, A_OUT2.4, IC5A.Y3
- removed net A_SWAP: A_OUT2.1, A_SWAP.C, IC5A.Y0
- removed net BUS0: BACKBUS.1, IC4A.A, IC5A.A
- removed net BUS1: BACKBUS.2, IC4A.B, IC5A.B
- removed net BUS10: BACKBUS.11, C_IN.C, C_REG.1
- removed net BUS11: BACKBUS.12, D_IN.C, D_REG.1
- removed net BUS12: BACKBUS.13, X_IN.C, X_REG.1
- removed net BUS13: BACKBUS.14, IR_IN.C, RAN_IN_3.2
- removed net BUS14: BACKBUS.15, MAR_IN.C, RAN_IN_3.1
- removed net BUS15: BACKBUS.16, PC_IN.C, RAN_IN_2.4
- removed net BUS16: FRONTBUS.1, RAM_IN_LOW.C, RAN_IN_2.3
- removed net BUS17: FRONTBUS.2, RAM_IN_H.C, RAN_IN_2.2
- removed net BUS18: FRONTBUS.3, IC3A.A
- removed net BUS19: FRONTBUS.4, IC3A.B
- removed net BUS2: BACKBUS.3, IC4A.C, IC5A.C
- removed net BUS20: FRONTBUS.5, IC3A.C
- removed net BUS21: FRONTBUS.6, PC_INC.C, RAN_IN_2.1
- removed net BUS22: FRONTBUS.7, STACK.2, STACK_INC.C
- removed net BUS23: FRONTBUS.8, STACK.3, STACK_DEC.C
- removed net BUS24: C_INC.C, C_REG.2, FRONTBUS.9
- removed net BUS25: C_DEC.C, C_REG.3, FRONTBUS.10
- removed net BUS26: FRONTBUS.11, RAN_IN_1.3, RESET.C
- removed net BUS27: FRONTBUS.12, HALT.C, RAN_IN_1.2
- removed net BUS28: FRONTBUS.13, NEXT_INS.C, RAN_IN_1.1
- removed net BUS29: FRONTBUS.14, STACK.1, STACK_IN.C
- removed net BUS3: BACKBUS.4, IC4A.G2A, IC5A.G2A
- removed net BUS30: FRONTBUS.15
- removed net BUS31: FRONTBUS.16
- removed net BUS4: BACKBUS.5, IC14A.A
- removed net BUS5: BACKBUS.6, IC14A.B
- removed net BUS6: BACKBUS.7, IC14A.C
- removed net BUS7: BACKBUS.8, IC1A.A
- removed net BUS8: BACKBUS.9, IC1A.B
- removed net BUS9: BACKBUS.10, IC1A.C
- removed net B_CLEAR: B_CLEAR.C, B_IN_LOW.4, IC1A.Y0
- removed net B_HIGH: B_HIGH.C, B_OUT2.2, IC5A.Y5
- removed net B_IN: B_IN.C, B_IN_LOW.3, IC1A.Y1
- removed net B_IN_H_H: B_IN_H_H.C, B_IN_LOW.1, IC1A.Y3
- removed net B_IN_H_L: B_IN_HIGH.1, B_IN_H_L.C, IC1A.Y5
- removed net B_IN_L_H: B_IN_HIGH.2, B_IN_L_H.C, IC1A.Y4
- removed net B_IN_L_L: B_IN_LOW.2, B_IN_L_L.C, IC1A.Y2
- removed net B_LOW: B_LOW.C, B_OUT2.3, IC5A.Y6
- removed net B_OUT: B_OUT.C, B_OUT2.4, IC5A.Y7
- removed net B_SWAP: B_OUT2.1, B_SWAP.C, IC5A.Y4
- removed net HALT_LED: NEXT_INS.A, R3.13
- removed net NOT: ALU_HIGH.1, IC3A.Y4, NOT.C
- removed net OR: ALU_HIGH.2, IC3A.Y5, OR.C
- removed net PC_OUT: IC4A.Y1, PC_OUT.C
- removed net RAM_OUT: IC4A.Y6, RAM_OUT.C
- removed net SHL: ALU_LOW.3, IC3A.Y2, SHL.C
- removed net SHR: ALU_LOW.4, IC3A.Y3, SHR.C
- removed net SUB: ALU_LOW.2, IC3A.Y1, SUB.C
- removed net XOR: ALU_HIGH.4, IC3A.Y7, XOR.C
- new net A: IC27.(ADC0)PA0, RN2A.2
- new net B: IC27.(ADC1)PA1, RN2B.2
- new net BANKA_PROG: BANKA.!WE, JP4.5, R12.1
- new net BANKB_PROG: BANKB.!WE, JP4.3, R13.1
- new net BANKC_PROG: BANKC.!WE, JP4.1, R14.1
- new net C: IC27.(ADC2)PA2, RN2C.2
- new net D: IC27.(ADC3)PA3, RN2D.2
- new net DIG0: IC27.(T0/XCK)PB0, U$1.DIG1
- new net DIG1: IC27.(T1)PB1, U$1.DIG2
- new net DIG2: IC27.(AIN0/INT2)PB2, U$1.DIG3
- new net DIG3: IC27.(AIN1/OC0)PB3, U$1.DIG4
- new net DP: IC27.(ADC7)PA7, RN2H.2
- new net E: IC27.(ADC4)PA4, RN2E.2
- new net EXTERN_BUS0: IC27.(RXD)PD0, R10.1, SV3.1
- new net EXTERN_BUS1: IC27.(TXD)PD1, R10.9, SV3.2
- new net EXTERN_BUS10: IC27.PC2, R10.6, SV3.11
- new net EXTERN_BUS11: IC27.PC3, R10.14, SV3.12
- new net EXTERN_BUS12: IC27.PC4, R10.7, SV3.13
- new net EXTERN_BUS13: IC27.PC5, R10.15, SV3.14
- new net EXTERN_BUS14: IC27.(TOSC1)PC6, R10.8, SV3.15
- new net EXTERN_BUS15: IC27.(TOSC2)PC7, PULL_DOWN.1, SV3.16
- new net EXTERN_BUS2: IC27.(INT0)PD2, R10.2, SV3.3
- new net EXTERN_BUS3: IC27.(INT1)PD3, R10.10, SV3.4
- new net EXTERN_BUS4: IC27.(OC1B)PD4, R10.3, SV3.5
- new net EXTERN_BUS5: IC27.(OC1A)PD5, R10.11, SV3.6
- new net EXTERN_BUS6: IC27.(ICP)PD6, R10.4, SV3.7
- new net EXTERN_BUS7: IC27.(OC2)PD7, R10.12, SV3.8
- new net EXTERN_BUS8: IC27.PC0(SCL), R10.5, SV3.9
- new net EXTERN_BUS9: IC27.PC1(SDA), R10.13, SV3.10
- new net F: IC27.(ADC5)PA5, RN2F.2
- new net G: IC27.(ADC6)PA6, RN2G.2
- new net N$100: D_OUT.A, R3.14
- new net N$101: D_LOW.A, R3.13
- new net N$102: D_HIGH.A, R3.12
- new net N$103: D_SWAP.A, R3.11
- new net N$104: R3.10, X_OUT.A
- new net N$105: PC_OUT.A, R3.9
- new net N$106: IC5A.Y0, RAM_IMT_OUT.1, RAM_OUT.C
- new net N$107: IC5A.Y1, INTERUPT_OUT.C, RAM_IMT_OUT.2
- new net N$108: EXTRA_OUT.4, EXTRA_OUT1.C, IC5A.Y2
- new net N$109: EXTRA_OUT.3, EXTRA_OUT2.C, IC5A.Y3
- new net N$110: EXTRA_OUT.2, EXTRA_OUT3.C, IC5A.Y4
- new net N$111: EXTRA_OUT.1, EXTRA_OUT4.C, IC5A.Y5
- new net N$112: R2.1, STACK_OUT.A
- new net N$113: EXTRA_OUT4.A, R2.8
- new net N$114: EXTRA_OUT3.A, R2.7
- new net N$115: EXTRA_OUT2.A, R2.6
- new net N$116: EXTRA_OUT1.A, R2.5
- new net N$117: R2.2, RAM_OUT.A
- new net N$118: INTERUPT_OUT.A, R2.3
- new net N$119: IC27.(MOSI)PB5, SV5.3
- new net N$120: IC27.(SCK)PB7, SV5.4
- new net N$121: IC27.(MISO)PB6, SV5.6
- new net N$122: IC27.RESET, SV5.2
- new net N$123: RN2A.1, U$1.A
- new net N$124: RN2B.1, U$1.B
- new net N$125: RN2C.1, U$1.C
- new net N$126: RN2D.1, U$1.D
- new net N$127: RN2E.1, U$1.E
- new net N$128: RN2F.1, U$1.F
- new net N$129: RN2G.1, U$1.G
- new net N$130: RN2H.1, U$1.DP
- new net N$131: R2.15, STEP1.A
- new net N$132: R2.14, STEP2.A
- new net N$133: R2.13, STEP3.A
- new net N$134: R2.12, STEP4.A
- new net N$37: BANKA.VSS, BANKA.VSS2, BANKB.VSS, BANKB.VSS2, BANKC.VSS, BANKC.VSS2
- new net N$42: BANKA.!OE, BANKB.!OE, BANKC.!OE, READ_WRITE.2
- new net N$43: EXTRA5.A, R8.5
- new net N$63: IC1A.Y2, SHIFT_ROLL.4, SHL.C
- new net N$64: IC1A.Y3, SHIFT_ROLL.3, SHR.C
- new net N$65: IC1A.Y4, ROL.C, SHIFT_ROLL.2
- new net N$66: IC1A.Y5, ROR.C, SHIFT_ROLL.1
- new net N$67: NOT.A, R7.9
- new net N$68: AND.A, R7.10
- new net N$69: OR.A, R7.11
- new net N$70: R7.12, XOR.A
- new net N$71: IC23A.Y7, LOGIC_OP.1, XOR.C
- new net N$72: IC23A.Y6, LOGIC_OP.2, OR.C
- new net N$73: AND.C, IC23A.Y5, LOGIC_OP.3
- new net N$74: IC23A.Y4, LOGIC_OP.4, NOT.C
- new net N$75: A_OUT.C, A_OUT_PINS.1, IC3A.Y0
- new net N$76: A_LOW.C, A_OUT_PINS.2, IC3A.Y1
- new net N$77: A_HIGH.C, A_OUT_PINS.3, IC3A.Y2
- new net N$78: A_OUT_PINS.4, A_SWAP.C, IC3A.Y3
- new net N$79: B_OUT.C, B_OUT_PIMS.1, IC3A.Y4
- new net N$80: B_LOW.C, B_OUT_PIMS.2, IC3A.Y5
- new net N$81: B_HIGH.C, B_OUT_PIMS.3, IC3A.Y6
- new net N$82: B_OUT_PIMS.4, B_SWAP.C, IC3A.Y7
- new net N$83: D_OUT.C, D_OUT_PINS.1, IC4A.Y1
- new net N$84: C_OUT.C, C_X_OC_STACK_OUT.4, IC4A.Y0
- new net N$85: D_LOW.C, D_OUT_PINS.2, IC4A.Y2
- new net N$86: D_HIGH.C, D_OUT_PINS.3, IC4A.Y3
- new net N$87: D_OUT_PINS.4, D_SWAP.C, IC4A.Y4
- new net N$88: C_X_OC_STACK_OUT.3, IC4A.Y5, X_OUT.C
- new net N$89: C_X_OC_STACK_OUT.2, IC4A.Y6, PC_OUT.C
- new net N$90: C_X_OC_STACK_OUT.1, IC4A.Y7, STACK_OUT.C
- new net N$91: A_OUT.A, R3.1
- new net N$92: A_LOW.A, R3.2
- new net N$93: A_HIGH.A, R3.3
- new net N$94: A_SWAP.A, R3.4
- new net N$95: B_OUT.A, R3.5
- new net N$96: B_LOW.A, R3.6
- new net N$97: B_HIGH.A, R3.7
- new net N$98: B_SWAP.A, R3.8
- new net N$99: C_OUT.A, R3.15
- new net WRITE_ENABLE: BANKA.!WP, BANKB.!WP, BANKC.!WP, JP3.2
- net !CLEAR: now also BANKA.!RST, BANKB.!RST, BANKC.!RST, CLEAR_OUNS.1; no longer JP4.1
- net ADDR_BUS0: now also BANKA.A0; no longer U$1.A0
- net ADDR_BUS1: now also BANKA.A1; no longer U$1.A1
- net ADDR_BUS10: now also BANKA.A10; no longer U$1.A10
- net ADDR_BUS11: now also BANKA.A11; no longer U$1.A11
- net ADDR_BUS12: now also BANKA.A12; no longer U$1.A12
- net ADDR_BUS13: now also BANKA.A13; no longer U$1.A13
- net ADDR_BUS14: now also BANKA.A14; no longer U$1.A14
- net ADDR_BUS15: now also BANKA.A15; no longer U$1.A15
- net ADDR_BUS16: now also BANKA.A16; no longer U$1.A16
- net ADDR_BUS17: now also BANKA.A17; no longer U$1.A17
- net ADDR_BUS18: now also BANKA.A18; no longer U$1.A18
- net ADDR_BUS19: now also BANKA.A19; no longer U$1.A19
- net ADDR_BUS2: now also BANKA.A2; no longer U$1.A2
- net ADDR_BUS3: now also BANKA.A3; no longer U$1.A3
- net ADDR_BUS4: now also BANKA.A4; no longer U$1.A4
- net ADDR_BUS5: now also BANKA.A5; no longer U$1.A5
- net ADDR_BUS6: now also BANKA.A6; no longer U$1.A6
- net ADDR_BUS7: now also BANKA.A7; no longer U$1.A7
- net ADDR_BUS8: now also BANKA.A8; no longer U$1.A8
- net ADDR_BUS9: now also BANKA.A9; no longer U$1.A9
- net CLEAR: now also CLEAR_OUNS.2; no longer JP4.2
- net DATAA0: now also BANKA.DQ0, IC3A.A, IC4A.A, IC5A.A; no longer U$1.DQ0
- net DATAA1: now also BANKA.DQ1, IC3A.B, IC4A.B, IC5A.B; no longer U$1.DQ1
- net DATAA10: now also BANKA.DQ10, EXTRA6.C, EXTRA_5_6_PINS.2; no longer U$1.DQ10
- net DATAA11: now also ABC_CLEAR.1, A_CLEAR_LED.C, BANKA.DQ11; no longer U$1.DQ11
- net DATAA12: now also ABC_CLEAR.2, BANKA.DQ12, B_CLEAR_LED.C; no longer U$1.DQ12
- net DATAA13: now also ABC_CLEAR.3, BANKA.DQ13, D_CLEAR_LED.C; no longer U$1.DQ13
- net DATAA14: now also BANKA.DQ14, INTERUPTS.1, PAUSE_INERUPT.C; no longer U$1.DQ14
- net DATAA15: now also BANKA.DQ15, INTERUPTS.2, PLAY_INTERUPT.C; no longer U$1.DQ15
- net DATAA2: now also BANKA.DQ2, IC3A.C, IC4A.C, IC5A.C; no longer U$1.DQ2
- net DATAA3: now also BANKA.DQ3, IC3A.G2A, IC4A.G2A, IC5A.G2A; no longer U$1.DQ3
- net DATAA4: now also BANKA.DQ4, IC3A.G2B, IC4A.G2B, IC5A.G2B; no longer U$1.DQ4
- net DATAA5: now also BANKA.DQ5, EXTRA1.C, EXTRA_1_2_PINS.1; no longer U$1.DQ5
- net DATAA6: now also BANKA.DQ6, EXTRA2.C, EXTRA_1_2_PINS.2; no longer U$1.DQ6
- net DATAA7: now also BANKA.DQ7, EXTRA3.C, EXTRA_3_4_PINS.1; no longer U$1.DQ7
- net DATAA8: now also BANKA.DQ8, EXTRA4.C, EXTRA_3_4_PINS.2; no longer U$1.DQ8
- net DATAA9: now also BANKA.DQ9, EXTRA5.C, EXTRA_5_6_PINS.1; no longer U$1.DQ9
- net DATAB0: now also IC21A.A
- net DATAB1: now also IC21A.B
- net DATAB10: now also IR_IN.C, PC_MAR_IR_IN.1
- net DATAB11: now also MAR_IN.C, PC_MAR_IR_IN.2
- net DATAB12: now also PC_IN.C, PC_MAR_IR_IN.3
- net DATAB13: now also RAM_STACK_IN.1, STACK_IN.C
- net DATAB14: now also RAM_IN_L.C, RAM_STACK_IN.2
- net DATAB15: now also RAM_IN_H.C, RAM_STACK_IN.3
- net DATAB2: now also IC21A.C
- net DATAB3: now also IC22A.A
- net DATAB4: now also IC22A.B, PC_INC_DEC.2
- net DATAB5: now also IC22A.C
- net DATAB6: now also C_IN.C, IN_C_D_X.1
- net DATAB7: now also D_IN_L.C, IN_C_D_X.2
- net DATAB8: now also D_IN_H.C, IN_C_D_X.3
- net DATAB9: now also IN_C_D_X.4, X_IN.C
- net DATAC0: now also IC1A.A, IC23A.A
- net DATAC1: now also IC1A.B, IC23A.B
- net DATAC13: now also HALT_RESEDT_NEXTINS.3, RESET.C
- net DATAC14: now also HALT.C, HALT_RESEDT_NEXTINS.2
- net DATAC15: now also HALT_RESEDT_NEXTINS.1, NEXT_INS.C
- net DATAC2: now also IC1A.C, IC23A.C
- net DATAC3: now also IC1A.G2A, IC23A.G2A
- net DATAC4: now also PC_DEC.C
- net DATAC5: now also PC_INC.C, PC_INC_DEC.1
- net DATAC6: now also STACK_C.4, STACK_INC.C
- net DATAC7: now also STACK_C.3, STACK_DEC.C
- net DATAC8: now also C_INC.C, STACK_C.2
- net DATAC9: now also C_DEC.C, STACK_C.1
- net GND: now also BANKA.!CE, BANKA.VDD, BANKB.!CE, BANKB.VDD, BANKC.!CE, BANKC.VDD, IC21A.G2A, IC21A.G2B, IC22A.G2A, IC22A.G2B, IC23A.G2B, IC27.AREF, IC27.GND, IC27.GND1, IC27.GND2, IC27.GND@1, PULL_DOWN.2, R10.16, READ_WRITE.3, SV5.1; no longer IC14A.G2A, IC14A.G2B, IC1A.G2A, IC3A.G2A, IC3A.G2B, IC4A.G2B, IC5A.G2B
- net IN_BUS0: now also STEP1.C, STEP_PINS.1
- net IN_BUS1: now also STEP2.C, STEP_PINS.2
- net IN_BUS2: now also STEP3.C, STEP_PINS.3
- net IN_BUS3: now also STEP4.C, STEP_PINS.4
- net N$10: now also D_CLEAR_LED.A, R8.9; no longer IC4A.Y4, X_REG.2, X_SWAP.C
- net N$11: now also PAUSE_INERUPT.A, R8.10; no longer R3.2, X_IN.A
- net N$12: now also PLAY_INTERUPT.A, R8.11; no longer IC4A.Y7, X_OUT.C, X_REG.3
- net N$13: now also C_IN.A, R8.12; no longer R3.15, X_OUT.A
- net N$14: now also D_IN_L.A, R8.15; no longer R3.9, STACK_IN.A
- net N$15: now also D_IN_H.A, R8.14; no longer R3.10, STACK_INC.A
- net N$16: now also PC_INC.A, R5.1; no longer R3.11, STACK_DEC.A
- net N$17: now also PC_DEC.A, R5.2; no longer R3.12, STACK_OUT.A
- net N$18: now also IR_IN.A, R5.3; no longer IC4A.Y2, STACK.4, STACK_OUT.C
- net N$19: now also MAR_IN.A, R5.4; no longer D_REG.2, D_SWAP.C, IC4A.Y0
- net N$2: now also EXTRA1.A, R8.1; no longer C_IN.A, R3.8
- net N$20: now also PC_IN.A, R5.5; no longer D_SWAP.A, R3.14
- net N$21: now also R5.6, STACK_IN.A; no longer A_CLEAR.A, R5.9
- net N$22: now also R5.7, RAM_IN_L.A; no longer ADD.A, R5.1
- net N$23: now also R5.8, RAM_IN_H.A; no longer A_IN.A, R5.10
- net N$24: now also NEXT_INS.A, R5.10; no longer B_CLEAR.A, R4.9
- net N$25: now also R5.15, STACK_DEC.A; no longer B_IN.A, R4.10
- net N$26: now also C_INC.A, R5.14; no longer B_IN_L_L.A, R4.11
- net N$27: now also C_DEC.A, R5.13; no longer B_IN_H_H.A, R4.12
- net N$28: now also R5.12, RESET.A; no longer R5.8, XOR.A
- net N$29: now also HALT.A, R5.11; no longer AND.A, R5.7
- net N$3: now also EXTRA2.A, R8.2; no longer C_OUT.C, C_REG.4, IC4A.Y5
- net N$30: now also R5.9, STACK_INC.A; no longer OR.A, R5.6
- net N$31: now also A_IN.C, A_IN_LOW.1, IC21A.Y0; no longer NOT.A, R5.5
- net N$32: now also A_IN_LOW.2, A_IN_L_L.C, IC21A.Y1; no longer R5.4, SHR.A
- net N$33: now also A_IN_H_H.C, A_IN_LOW.3, IC21A.Y2; no longer R5.3, SHL.A
- net N$34: now also A_IN_HIGH.1, A_IN_L_H.C, IC21A.Y3; no longer R5.2, SUB.A
- net N$35: now also A_IN_HIGH.2, A_IN_H_L.C, IC21A.Y4; no longer B_IN_L_H.A, R4.13
- net N$36: now also A_IN.A, R4.8; no longer B_IN_H_L.A, R4.14
- net N$38: now also R4.7; no longer R5.11
- net N$39: now also R4.6; no longer R5.12
- net N$4: now also R8.13, X_IN.A; no longer C_OUT.A, R3.5
- net N$40: now also R4.5; no longer R5.13
- net N$41: now also R4.4; no longer R5.14
- net N$44: now also B_IN.A, B_IN_LOW1.3, IC22A.Y0; no longer R2.15, RAM_OUT.A, RAM_PC_OUT.2
- net N$45: now also B_IN_LOW1.2, B_IN_L_L.A, IC22A.Y1; no longer A_SWAP.A, R2.1
- net N$46: now also B_IN_H_H.A, B_IN_LOW1.1, IC22A.Y2; no longer A_HIGH.A, R2.2
- net N$47: now also B_IN_HIGH1.2, B_IN_L_H.A, IC22A.Y3; no longer A_LOW.A, R2.3
- net N$48: now also B_IN_HIGH1.1, B_IN_H_L.A, IC22A.Y4; no longer A_OUT.A, R2.4
- net N$49: now also B_IN.C, R4.9; no longer B_SWAP.A, R2.5
- net N$5: now also EXTRA4.A, R8.4; no longer C_DEC.A, R3.6
- net N$51: now also B_IN_L_L.C, R4.10; no longer B_HIGH.A, R2.6
- net N$52: now also B_IN_H_H.C, R4.11; no longer B_LOW.A, R2.7
- net N$53: now also B_IN_L_H.C, R4.12; no longer B_OUT.A, R2.8
- net N$54: now also B_IN_H_L.C, R4.14; no longer PC_OUT.A, R2.14, RAM_PC_OUT.1
- net N$55: now also R7.8, ROR.A; no longer IR_IN.A, R4.8
- net N$56: now also R7.7, ROL.A; no longer MAR_IN.A, R4.7
- net N$57: now also R7.6, SHR.A; no longer PC_IN.A, R4.6
- net N$58: now also R7.5, SHL.A; no longer R4.5, RAM_IN_LOW.A
- net N$59: now also R7.4, SUB.A; no longer R4.4, RAM_IN_H.A
- net N$6: now also EXTRA3.A, R8.3; no longer C_INC.A, R3.7
- net N$60: now also ADD.A, R7.3; no longer PC_INC.A, R4.3
- net N$61: now also ADD.C, ADD_SUB.2, IC1A.Y0; no longer R4.2, RESET.A
- net N$62: now also ADD_SUB.1, IC1A.Y1, SUB.C; no longer HALT.A, R4.1
- net N$7: now also EXTRA6.A, R8.6; no longer D_OUT.A, D_OUT.C, D_REG.3, IC4A.Y3, R3.3
- net N$8: now also B_CLEAR_LED.A, R8.8; no longer D_IN.A, R3.4
- net N$9: now also A_CLEAR_LED.A, R8.7; no longer R3.1, X_SWAP.A
- net PROGRAM: now also JP4.2, JP4.4, JP4.6
- net VCC: now also IC21A.G1, IC22A.G1, IC23A.G1, IC27.AVCC, IC27.VCC, IC27.VCC1, IC27.VCC2, R12.2, R13.2, R14.2, R7.16, R8.16, READ_WRITE.1, SV5.5; no longer IC14A.G1

Commit message: Controller done?
Parts:
- removed ADD_HIGH, ADD_LOW, ADD_MID, BA_HIGH, BA_LOW, BB_HIGH, BB_LOW, BC_HIGH, BC_LOW: 74ABT164D, 74xx-us:74ABT164D
- removed JP4: (no value), jumper:JP3Q
- removed R12, R13, R14: (no value), rcl:R-US_M0805
- removed READ_WRITE: (no value), jumper:JP2E
- removed SW_PROD_1, SW_PROD_2, SW_PROD_3, SW_PROD_4, SW_PROD_5: 74LS157D, 74xx-us:74LS157D
- added SV2: (no value), con-harting-ml:ML6
- BANKA, BANKB, BANKC: value SST39VF1602-70-4I-EKE -> (none); device 16bit:SST39VF1602-70-4I-EKE -> con-harting-ml:ML16
- JP3: device jumper:JP6Q -> pinhead:PINHD-1X20
Connections:
- removed net ADDR_BUS0: BANKA.A0, BANKB.A0, BANKC.A0, SW_PROD_1A.4Y
- removed net ADDR_BUS1: BANKA.A1, BANKB.A1, BANKC.A1, SW_PROD_1A.3Y
- removed net ADDR_BUS10: BANKA.A10, BANKB.A10, BANKC.A10, SW_PROD_3A.2Y
- removed net ADDR_BUS11: BANKA.A11, BANKB.A11, BANKC.A11, SW_PROD_3A.1Y
- removed net ADDR_BUS12: BANKA.A12, BANKB.A12, BANKC.A12, SW_PROD_4A.1Y
- removed net ADDR_BUS13: BANKA.A13, BANKB.A13, BANKC.A13, SW_PROD_4A.2Y
- removed net ADDR_BUS14: BANKA.A14, BANKB.A14, BANKC.A14, SW_PROD_4A.3Y
- removed net ADDR_BUS15: BANKA.A15, BANKB.A15, BANKC.A15, SW_PROD_4A.4Y
- removed net ADDR_BUS16: BANKA.A16, BANKB.A16, BANKC.A16, SW_PROD_5A.1Y
- removed net ADDR_BUS17: BANKA.A17, BANKB.A17, BANKC.A17, SW_PROD_5A.2Y
- removed net ADDR_BUS18: BANKA.A18, BANKB.A18, BANKC.A18, SW_PROD_5A.3Y
- removed net ADDR_BUS19: BANKA.A19, BANKB.A19, BANKC.A19, SW_PROD_5A.4Y
- removed net ADDR_BUS2: BANKA.A2, BANKB.A2, BANKC.A2, SW_PROD_1A.2Y
- removed net ADDR_BUS3: BANKA.A3, BANKB.A3, BANKC.A3, SW_PROD_1A.1Y
- removed net ADDR_BUS4: BANKA.A4, BANKB.A4, BANKC.A4, SW_PROD_2A.4Y
- removed net ADDR_BUS5: BANKA.A5, BANKB.A5, BANKC.A5, SW_PROD_2A.3Y
- removed net ADDR_BUS6: BANKA.A6, BANKB.A6, BANKC.A6, SW_PROD_2A.2Y
- removed net ADDR_BUS7: BANKA.A7, BANKB.A7, BANKC.A7, SW_PROD_2A.1Y
- removed net ADDR_BUS8: BANKA.A8, BANKB.A8, BANKC.A8, SW_PROD_3A.4Y
- removed net ADDR_BUS9: BANKA.A9, BANKB.A9, BANKC.A9, SW_PROD_3A.3Y
- removed net ADDR_SHIFT: ADD_LOWA.A, ADD_LOWA.B, JP3.5
- removed net BANKA_PROG: BANKA.!WE, JP4.5, R12.1
- removed net BANKB_PROG: BANKB.!WE, JP4.3, R13.1
- removed net BANKC_PROG: BANKC.!WE, JP4.1, R14.1
- removed net DATAA_SHIFT: BA_LOWA.A, BA_LOWA.B, JP3.6
- removed net DATAB_SHIFT: BB_LOWA.A, BB_LOWA.B, JP3.4
- removed net DATAC_SHIFT: BC_LOWA.A, BC_LOWA.B, JP3.3
- removed net DATA_ADDR_CLOCK: BA_HIGHA.CLK, BA_LOWA.CLK, BB_HIGHA.CLK, BB_LOWA.CLK, BC_HIGHA.CLK, BC_LOWA.CLK, JP3.7
- removed net N$37: BANKA.VSS, BANKA.VSS2, BANKB.VSS, BANKB.VSS2, BANKC.VSS, BANKC.VSS2
- removed net N$42: BANKA.!OE, BANKB.!OE, BANKC.!OE, READ_WRITE.2
- removed net PROGRAM: JP3.9, JP4.2, JP4.4, JP4.6
- removed net PROG_ADDR0: ADD_LOWA.QA, SW_PROD_1A.4B
- removed net PROG_ADDR1: ADD_LOWA.QB, SW_PROD_1A.3B
- removed net PROG_ADDR10: ADD_MIDA.QC, SW_PROD_3A.2B
- removed net PROG_ADDR11: ADD_MIDA.QD, SW_PROD_3A.1B
- removed net PROG_ADDR12: ADD_MIDA.QE, SW_PROD_4A.1B
- removed net PROG_ADDR13: ADD_MIDA.QF, SW_PROD_4A.2B
- removed net PROG_ADDR14: ADD_MIDA.QG, SW_PROD_4A.3B
- removed net PROG_ADDR15: ADD_HIGHA.A, ADD_HIGHA.B, ADD_MIDA.QH, SW_PROD_4A.4B
- removed net PROG_ADDR16: ADD_HIGHA.QA, SW_PROD_5A.1B
- removed net PROG_ADDR17: ADD_HIGHA.QB, SW_PROD_5A.2B
- removed net PROG_ADDR18: ADD_HIGHA.QC, SW_PROD_5A.3B
- removed net PROG_ADDR19: ADD_HIGHA.QD, SW_PROD_5A.4B
- removed net PROG_ADDR2: ADD_LOWA.QC, SW_PROD_1A.2B
- removed net PROG_ADDR3: ADD_LOWA.QD, SW_PROD_1A.1B
- removed net PROG_ADDR4: ADD_LOWA.QE, SW_PROD_2A.4B
- removed net PROG_ADDR5: ADD_LOWA.QF, SW_PROD_2A.3B
- removed net PROG_ADDR6: ADD_LOWA.QG, SW_PROD_2A.2B
- removed net PROG_ADDR7: ADD_LOWA.QH, ADD_MIDA.A, ADD_MIDA.B, SW_PROD_2A.1B
- removed net PROG_ADDR8: ADD_MIDA.QA, SW_PROD_3A.4B
- removed net PROG_ADDR9: ADD_MIDA.QB, SW_PROD_3A.3B
- removed net PROG_ADDR_CLOCK: ADD_HIGHA.CLK, ADD_LOWA.CLK, ADD_MIDA.CLK, JP3.8
- removed net PROG_CLEAR: ADD_HIGHA.CLR, ADD_LOWA.CLR, ADD_MIDA.CLR, BA_HIGHA.CLR, BA_LOWA.CLR, BB_HIGHA.CLR, BB_LOWA.CLR, BC_HIGHA.CLR, BC_LOWA.CLR, JP3.10
- removed net PROG_DIR: JP3.1, SW_PROD_1A.!A!/B, SW_PROD_2A.!A!/B, SW_PROD_3A.!A!/B, SW_PROD_4A.!A!/B, SW_PROD_5A.!A!/B
- removed net WRITE_ENABLE: BANKA.!WP, BANKB.!WP, BANKC.!WP, JP3.2
- net !CLEAR: no longer BANKA.!RST, BANKB.!RST, BANKC.!RST
- net DATAA0: now also BANKA.1; no longer BANKA.DQ0, BA_LOWA.QA
- net DATAA1: now also BANKA.2; no longer BANKA.DQ1, BA_LOWA.QB
- net DATAA10: now also BANKA.11; no longer BANKA.DQ10, BA_HIGHA.QC
- net DATAA11: now also BANKA.12; no longer BANKA.DQ11, BA_HIGHA.QD
- net DATAA12: now also BANKA.13; no longer BANKA.DQ12, BA_HIGHA.QE
- net DATAA13: now also BANKA.14; no longer BANKA.DQ13, BA_HIGHA.QF
- net DATAA14: now also BANKA.15; no longer BANKA.DQ14, BA_HIGHA.QG
- net DATAA15: now also BANKA.16; no longer BANKA.DQ15, BA_HIGHA.QH
- net DATAA2: now also BANKA.3; no longer BANKA.DQ2, BA_LOWA.QC
- net DATAA3: now also BANKA.4; no longer BANKA.DQ3, BA_LOWA.QD
- net DATAA4: now also BANKA.5; no longer BANKA.DQ4, BA_LOWA.QE
- net DATAA5: now also BANKA.6; no longer BANKA.DQ5, BA_LOWA.QF
- net DATAA6: now also BANKA.7; no longer BANKA.DQ6, BA_LOWA.QG
- net DATAA7: now also BANKA.8; no longer BANKA.DQ7, BA_HIGHA.A, BA_HIGHA.B, BA_LOWA.QH
- net DATAA8: now also BANKA.9; no longer BANKA.DQ8, BA_HIGHA.QA
- net DATAA9: now also BANKA.10; no longer BANKA.DQ9, BA_HIGHA.QB
- net DATAB0: now also BANKB.1; no longer BANKB.DQ0, BB_LOWA.QA
- net DATAB1: now also BANKB.2; no longer BANKB.DQ1, BB_LOWA.QB
- net DATAB10: now also BANKB.11; no longer BANKB.DQ10, BB_HIGHA.QC
- net DATAB11: now also BANKB.12; no longer BANKB.DQ11, BB_HIGHA.QD
- net DATAB12: now also BANKB.13; no longer BANKB.DQ12, BB_HIGHA.QE
- net DATAB13: now also BANKB.14; no longer BANKB.DQ13, BB_HIGHA.QF
- net DATAB14: now also BANKB.15; no longer BANKB.DQ14, BB_HIGHA.QG
- net DATAB15: now also BANKB.16; no longer BANKB.DQ15, BB_HIGHA.QH
- net DATAB2: now also BANKB.3; no longer BANKB.DQ2, BB_LOWA.QC
- net DATAB3: now also BANKB.4; no longer BANKB.DQ3, BB_LOWA.QD
- net DATAB4: now also BANKB.5; no longer BANKB.DQ4, BB_LOWA.QE
- net DATAB5: now also BANKB.6; no longer BANKB.DQ5, BB_LOWA.QF
- net DATAB6: now also BANKB.7; no longer BANKB.DQ6, BB_LOWA.QG
- net DATAB7: now also BANKB.8; no longer BANKB.DQ7, BB_HIGHA.A, BB_HIGHA.B, BB_LOWA.QH
- net DATAB8: now also BANKB.9; no longer BANKB.DQ8, BB_HIGHA.QA
- net DATAB9: now also BANKB.10; no longer BANKB.DQ9, BB_HIGHA.QB
- net DATAC0: now also BANKC.1; no longer BANKC.DQ0, BC_LOWA.QA
- net DATAC1: now also BANKC.2; no longer BANKC.DQ1, BC_LOWA.QB
- net DATAC10: now also BANKC.11; no longer BANKC.DQ10, BC_HIGHA.QC
- net DATAC11: now also BANKC.12; no longer BANKC.DQ11, BC_HIGHA.QD
- net DATAC12: now also BANKC.13; no longer BANKC.DQ12, BC_HIGHA.QE
- net DATAC13: now also BANKC.14; no longer BANKC.DQ13, BC_HIGHA.QF
- net DATAC14: now also BANKC.15; no longer BANKC.DQ14, BC_HIGHA.QG
- net DATAC15: now also BANKC.16; no longer BANKC.DQ15, BC_HIGHA.QH
- net DATAC2: now also BANKC.3; no longer BANKC.DQ2, BC_LOWA.QC
- net DATAC3: now also BANKC.4; no longer BANKC.DQ3, BC_LOWA.QD
- net DATAC4: now also BANKC.5; no longer BANKC.DQ4, BC_LOWA.QE
- net DATAC5: now also BANKC.6; no longer BANKC.DQ5, BC_LOWA.QF
- net DATAC6: now also BANKC.7; no longer BANKC.DQ6, BC_LOWA.QG
- net DATAC7: now also BANKC.8; no longer BANKC.DQ7, BC_HIGHA.A, BC_HIGHA.B, BC_LOWA.QH
- net DATAC8: now also BANKC.9; no longer BANKC.DQ8, BC_HIGHA.QA
- net DATAC9: now also BANKC.10; no longer BANKC.DQ9, BC_HIGHA.QB
- net GND: now also SV2.2, SV2.3; no longer BANKA.!CE, BANKA.VDD, BANKB.!CE, BANKB.VDD, BANKC.!CE, BANKC.VDD, JP3.11, READ_WRITE.3, SW_PROD_1A.G, SW_PROD_2A.G, SW_PROD_3A.G, SW_PROD_4A.G, SW_PROD_5A.G
- net IN_BUS0: now also JP3.20; no longer SW_PROD_1A.4A
- net IN_BUS1: now also JP3.10; no longer SW_PROD_1A.3A
- net IN_BUS10: now also JP3.15; no longer SW_PROD_3A.2A
- net IN_BUS11: now also JP3.5; no longer SW_PROD_3A.1A
- net IN_BUS12: now also JP3.14; no longer SW_PROD_4A.1A
- net IN_BUS13: now also JP3.4; no longer SW_PROD_4A.2A
- net IN_BUS14: now also JP3.13; no longer SW_PROD_4A.3A
- net IN_BUS15: now also JP3.3; no longer SW_PROD_4A.4A
- net IN_BUS16: now also JP3.12; no longer SW_PROD_5A.1A
- net IN_BUS17: now also JP3.2; no longer SW_PROD_5A.2A
- net IN_BUS18: now also JP3.11; no longer SW_PROD_5A.3A
- net IN_BUS19: now also JP3.1; no longer SW_PROD_5A.4A
- net IN_BUS2: now also JP3.19; no longer SW_PROD_1A.2A
- net IN_BUS3: now also JP3.9; no longer SW_PROD_1A.1A
- net IN_BUS4: now also JP3.18; no longer SW_PROD_2A.4A
- net IN_BUS5: now also JP3.8; no longer SW_PROD_2A.3A
- net IN_BUS6: now also JP3.17; no longer SW_PROD_2A.2A
- net IN_BUS7: now also JP3.7; no longer SW_PROD_2A.1A
- net IN_BUS8: now also JP3.16; no longer SW_PROD_3A.4A
- net IN_BUS9: now also JP3.6; no longer SW_PROD_3A.3A
- net VCC: now also SV2.1, SV2.4, SV2.5, SV2.6; no longer JP3.12, R12.2, R13.2, R14.2, READ_WRITE.1

Commit message: Finished All Boards
Parts:
- added C1, C2, C3, C4: 1uF, rcl:C-USC1206
Connections:
- net GND: now also C1.2, C2.2, C3.2, C4.2
- net VCC: now also C1.1, C2.1, C3.1, C4.1
