File: P1001-001 - 16bit CPU/P1001-001-007-320 - Programmer/P1001-001-003-320 - Controller.sch (EAGLE design)
At the start: 156 parts, among them IC1 74LS138D, IC10 74ALS00D, IC21 74LS138D, IC22 74LS138D, IC23 74LS138D, IC27 MEGA8535-A, IC3 74LS138D, IC4 74LS138D, IC5 74LS138D, J1 22-27-2041-04

Commit message: Controller done?
Parts:
- removed R6: (no value), resistor-bourns:2NBS16-15
- removed R9: (no value), rcl:R-US_M0805
- renumbered R11 to PULL_DOWN
Connections:
- new net N$43: EXTRA5.A, R8.5
- net DATAA10: no longer EXTRA5.A, R6.5, R8.5
- net N$10: no longer R6.9
- net N$11: no longer R6.10
- net N$12: no longer R6.11
- net N$13: no longer R6.12
- net N$14: no longer R6.15
- net N$15: no longer R6.14
- net N$2: no longer R6.1
- net N$3: no longer R6.2
- net N$4: no longer R6.13
- net N$5: no longer R6.4
- net N$6: no longer R6.3
- net N$7: no longer R6.6
- net N$8: no longer R6.8
- net N$9: no longer R6.7
- net VCC: no longer R6.16
