File: P1001-001 - 16bit CPU/P1001-001-007-320 - Programmer/P1001-001-007-320 - Programmer.brd (EAGLE design)
At the start: 200 x 48 mm, 17 parts, among them IC1 MEGA8535-A

Commit message: Check in the first try at soldering up the board
Changed lines of the file:
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@@
 <hole x="4" y="44" drill="0.12"/>
 <hole x="196" y="4" drill="0.12"/>
+<hole x="4" y="44" drill="3"/>
+<hole x="4" y="4" drill="3"/>
+<hole x="196" y="4" drill="3"/>
+<hole x="196" y="44" drill="3"/>
 </plain>
 <attributes>
