File: P1001-001 - 16bit CPU/P1001-001-004-320 - Register/BRD1001-001-004-320 - Register.brd (EAGLE design)
At the start: 200 x 48 mm, 16 parts, among them IC1 74HC173D, IC12 74AC245DW, IC2 74HC173D, IC27 MEGA8535-A, IC3 74HC173D, IC4 74HC173D, IC7 74AC245DW, J1 22-27-2041-04, J3 22-27-2041-04, J4 22-27-2061-06

Commit message: Finished All Boards
Parts:
- added C1, C2, C3, C4: 1uF, rcl:C1206
Connections:
- net GND: now also C1.2, C2.2, C3.2, C4.2
- net VCC: now also C1.1, C2.1, C3.1, C4.1
Routing:
- net VCC: track 256.5 -> 396.4 mm, vias 8 -> 16
- net GND: track 353.3 -> 409.6 mm, vias 16 -> 18
