File: P1001-001 - 16bit CPU/P1001-001-004-320 - Register/BRD1001-001-004-320 - Register.sch (EAGLE design)
At the start: 16 parts, among them IC1 74HC192D, IC12 74AC245DW, IC2 74HC192D, IC27 MEGA8535-A, IC3 74HC192D, IC4 74HC192D, IC5 74ALS04D, IC7 74AC245DW, J1 22-27-2041-04

Commit message: Added the simple reg, cleaned things up
Parts:
- removed IC5: 74ALS04D, 74xx-us:74ALS04D
- removed JP2: (no value), jumper:JP4E
- added J3: 22-27-2041-04, con-molex:22-27-2041-04
- added J4: 22-27-2061-06, con-molex:22-27-2061-06
- IC1, IC2, IC3, IC4: value 74HC192D -> 74HC173D; device 74xx-eu:74HC192D -> 74xx-eu:74HC173D
Connections:
- removed net !DEC: IC1A.DN, IC5C.O
- removed net !INC: IC1A.UP, IC5D.O
- removed net DEC: IC5C.I, JP2.2
- removed net IN: IC5B.I, JP2.1
- removed net INC: IC5D.I, JP2.3
- removed net N$1: IC4A.BO
- removed net N$2: IC1A.CO, IC2A.UP
- removed net N$3: IC1A.BO, IC2A.DN
- removed net N$4: IC2A.CO, IC3A.UP
- removed net N$5: IC2A.BO, IC3A.DN
- removed net N$6: IC3A.CO, IC4A.UP
- removed net N$7: IC3A.BO, IC4A.DN
- removed net OUT: IC5A.I, JP2.4
- net !REG_IN: now also IC1A.G1, IC1A.G2, IC2A.G1, IC2A.G2, IC3A.G1, IC3A.G2, IC4A.G1, IC4A.G2, J4-1.S; no longer IC1A.LD, IC2A.LD, IC3A.LD, IC4A.LD, IC5B.O
- net !REG_OUT: now also J3-1.S; no longer IC5A.O
- net BUS0: now also IC3A.D4; no longer IC1A.D
- net BUS1: now also IC3A.D3; no longer IC1A.C
- net BUS10: now also IC1A.D2; no longer IC3A.B
- net BUS11: now also IC1A.D1; no longer IC3A.A
- net BUS12: now also IC4A.D4; no longer IC4A.D
- net BUS13: now also IC4A.D3; no longer IC4A.C
- net BUS14: now also IC4A.D2; no longer IC4A.B
- net BUS15: now also IC4A.D1; no longer IC4A.A
- net BUS2: now also IC3A.D2; no longer IC1A.B
- net BUS3: now also IC3A.D1; no longer IC1A.A
- net BUS4: now also IC2A.D4; no longer IC2A.D
- net BUS5: now also IC2A.D3; no longer IC2A.C
- net BUS6: now also IC2A.D2; no longer IC2A.B
- net BUS7: now also IC2A.D1; no longer IC2A.A
- net BUS8: now also IC1A.D4; no longer IC3A.D
- net BUS9: now also IC1A.D3; no longer IC3A.C
- net CLEAR: now also J4-6.S; no longer J1-4.S
- net CLK: now also IC1A.CLK, IC2A.CLK, IC3A.CLK, IC4A.CLK
- net GND: now also IC1A.M, IC1A.N, IC2A.M, IC2A.N, IC3A.M, IC3A.N, IC4A.M, IC4A.N
- net SIGNAL0: now also IC3A.Q4; no longer IC1A.QD
- net SIGNAL1: now also IC3A.Q3; no longer IC1A.QC
- net SIGNAL10: now also IC1A.Q2; no longer IC3A.QB
- net SIGNAL11: now also IC1A.Q1; no longer IC3A.QA
- net SIGNAL12: now also IC4A.Q4; no longer IC4A.QD
- net SIGNAL13: now also IC4A.Q3; no longer IC4A.QC
- net SIGNAL14: now also IC4A.Q2; no longer IC4A.QB
- net SIGNAL15: now also IC4A.Q1; no longer IC4A.QA
- net SIGNAL2: now also IC3A.Q2; no longer IC1A.QB
- net SIGNAL3: now also IC3A.Q1; no longer IC1A.QA
- net SIGNAL4: now also IC2A.Q4; no longer IC2A.QD
- net SIGNAL5: now also IC2A.Q3; no longer IC2A.QC
- net SIGNAL6: now also IC2A.Q2; no longer IC2A.QB
- net SIGNAL7: now also IC2A.Q1; no longer IC2A.QA
- net SIGNAL8: now also IC1A.Q4; no longer IC3A.QD
- net SIGNAL9: now also IC1A.Q3; no longer IC3A.QC
Other:
- moved on the sheet: BACKBUS, FRONTBUS, J1-1, J1-2, J1-3

Commit message: Finished All Boards
Parts:
- added C1, C2, C3, C4: 1uF, rcl:C-USC1206
Connections:
- net GND: now also C1.2, C2.2, C3.2, C4.2
- net VCC: now also C1.1, C2.1, C3.1, C4.1
