File: P1001-001 - 16bit CPU/P1001-001-005-320 - Controller Flash/SCH1001-001-005-320 - Controller Flash.brd (EAGLE design)
At the start: 100 x 30 mm, 8 parts

Commit message: Finished All Boards
Connections:
- new net GND: JP1.5
- net VDD: no longer JP1.5
Changed lines of the file:
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@@
 </signal>
 <signal name="VDD">
-<contactref element="JP1" pad="5"/>
 <contactref element="U$1" pad="37"/>
 <contactref element="U$1" pad="26"/>
@@
 <wire x1="5.125" y1="10.125" x2="11.875" y2="16.875" width="0.1524" layer="1"/>
 <wire x1="5.125" y1="6.5" x2="5.125" y2="10.125" width="0.1524" layer="1"/>
-<wire x1="26.25" y1="24.125" x2="26.35" y2="24.19" width="0.1524" layer="16"/>
 <wire x1="60.75" y1="9.75" x2="59.625" y2="9.75" width="0.1524" layer="1"/>
 <wire x1="60.75" y1="14.75" x2="60.75" y2="9.75" width="0.1524" layer="16"/>
@@
 <via x="76.75" y="2" extent="1-16" drill="0.35"/>
 </signal>
+<signal name="GND">
+<contactref element="JP1" pad="5"/>
+</signal>
 </signals>
