File: P1001-001 - 16bit CPU/P1001-001-005-320 - Controller Flash/SCH1001-001-005-320 - Controller Flash.sch (EAGLE design)
At the start: 8 parts

Commit message: Finished All Boards
Connections:
- new net GND: JP1.5
- net VDD: no longer JP1.5
Changed lines of the file:
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@@
 <net name="VDD" class="0">
-<segment>
-<pinref part="JP1" gate="B" pin="5"/>
-<wire x1="81.28" y1="71.12" x2="96.52" y2="71.12" width="0.1524" layer="91"/>
-<label x="83.82" y="71.12" size="1.778" layer="95"/>
-</segment>
 <segment>
 <pinref part="U$1" gate="G$1" pin="VDD"/>
@@
 </segment>
 </net>
+<net name="GND" class="0">
+<segment>
+<pinref part="JP1" gate="B" pin="5"/>
+<wire x1="81.28" y1="71.12" x2="96.52" y2="71.12" width="0.1524" layer="91"/>
+<label x="83.82" y="71.12" size="1.778" layer="95"/>
+</segment>
+</net>
