File: P1001-001 - 16bit CPU/P1001-001-009-320 - ALU/SCH1001-001-009-320 - ALU.brd (EAGLE design)
At the start: 200 x 152 mm, 68 parts, among them IC14 74ALS04D, IC15 74ALS04D, IC16 74ALS04D, IC27 MEGA8535-A, IC42 74ALS04D, IC51 74LS173D, IC55 74ALS04D

Commit message: Finished All Boards
Parts:
- added C1, C2, C3, C4: 1uF, rcl:C1206
Connections:
- net GND: now also C1.2, C2.2, C3.2, C4.2
- net VCC: now also C1.1, C2.1, C3.1, C4.1
Routing:
- net VCC: track 1136.5 -> 1322.0 mm, vias 57 -> 65
- net GND: track 1171.5 -> 1267.2 mm, vias 71 -> 80
