File: P1001-001 - 16bit CPU/P1001-001-009-320 - ALU/SCH1001-001-009-320 - ALU.sch (EAGLE design)
At the start: 68 parts, among them IC14 74ALS04D, IC15 74ALS04D, IC16 74ALS04D, IC27 MEGA8535-A, IC42 74ALS04D, IC51 74LS173D, IC55 74ALS04D

Commit message: Finished All Boards
Parts:
- added C1, C2, C3, C4: 1uF, rcl:C-USC1206
Connections:
- net GND: now also C1.2, C2.2, C3.2, C4.2
- net VCC: now also C1.1, C2.1, C3.1, C4.1
Changed lines of the file:
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@@
 <part name="NOTA1" library="74xx-eu" library_urn="urn:adsk.eagle:library:85" deviceset="74*245" device="DW" package3d_urn="urn:adsk.eagle:package:2018/2" technology="AC"/>
 <part name="NOTA2" library="74xx-eu" library_urn="urn:adsk.eagle:library:85" deviceset="74*245" device="DW" package3d_urn="urn:adsk.eagle:package:2018/2" technology="AC"/>
+<part name="C3" library="rcl" library_urn="urn:adsk.eagle:library:334" deviceset="C-US" device="C1206" package3d_urn="urn:adsk.eagle:package:23618/2" value="1uF"/>
+<part name="C1" library="rcl" library_urn="urn:adsk.eagle:library:334" deviceset="C-US" device="C1206" package3d_urn="urn:adsk.eagle:package:23618/2" value="1uF"/>
+<part name="C2" library="rcl" library_urn="urn:adsk.eagle:library:334" deviceset="C-US" device="C1206" package3d_urn="urn:adsk.eagle:package:23618/2" value="1uF"/>
+<part name="C4" library="rcl" library_urn="urn:adsk.eagle:library:334" deviceset="C-US" device="C1206" package3d_urn="urn:adsk.eagle:package:23618/2" value="1uF"/>
 </parts>
 <sheets>
@@
 <attribute name="VALUE" x="-83.82" y="104.14" size="1.778" layer="96"/>
 </instance>
+<instance part="C3" gate="G$1" x="-93.98" y="88.9" smashed="yes" rot="R270">
+<attribute name="NAME" x="-93.345" y="87.884" size="1.778" layer="95" rot="R270"/>
+<attribute name="VALUE" x="-98.171" y="87.884" size="1.778" layer="96" rot="R270"/>
+</instance>
+<instance part="C1" gate="G$1" x="-93.98" y="81.28" smashed="yes" rot="R270">
+<attribute name="NAME" x="-93.345" y="80.264" size="1.778" layer="95" rot="R270"/>
+<attribute name="VALUE" x="-98.171" y="80.264" size="1.778" layer="96" rot="R270"/>
+</instance>
+<instance part="C2" gate="G$1" x="-93.98" y="73.66" smashed="yes" rot="R270">
+<attribute name="NAME" x="-93.345" y="72.644" size="1.778" layer="95" rot="R270"/>
+<attribute name="VALUE" x="-98.171" y="72.644" size="1.778" layer="96" rot="R270"/>
+</instance>
+<instance part="C4" gate="G$1" x="-93.98" y="66.04" smashed="yes" rot="R270">
+<attribute name="NAME" x="-93.345" y="65.024" size="1.778" layer="95" rot="R270"/>
+<attribute name="VALUE" x="-98.171" y="65.024" size="1.778" layer="96" rot="R270"/>
+</instance>
 </instances>
 <busses>
@@
 <wire x1="-93.98" y1="111.76" x2="-88.9" y2="111.76" width="0.1524" layer="91"/>
 <label x="-93.98" y="121.92" size="1.778" layer="95" rot="R90"/>
+</segment>
+<segment>
+<pinref part="C4" gate="G$1" pin="1"/>
+<wire x1="-91.44" y1="66.04" x2="-91.44" y2="73.66" width="0.1524" layer="91"/>
+<wire x1="-91.44" y1="73.66" x2="-91.44" y2="81.28" width="0.1524" layer="91"/>
+<wire x1="-91.44" y1="81.28" x2="-91.44" y2="88.9" width="0.1524" layer="91"/>
+<wire x1="-91.44" y1="88.9" x2="-91.44" y2="93.98" width="0.1524" layer="91"/>
+<wire x1="-91.44" y1="93.98" x2="-78.74" y2="93.98" width="0.1524" layer="91"/>
+<pinref part="C3" gate="G$1" pin="1"/>
+<junction x="-91.44" y="88.9"/>
+<pinref part="C1" gate="G$1" pin="1"/>
+<junction x="-91.44" y="81.28"/>
+<pinref part="C2" gate="G$1" pin="1"/>
+<junction x="-91.44" y="73.66"/>
+<label x="-86.36" y="93.98" size="1.778" layer="95"/>
 </segment>
 </net>
@@
 <label x="106.68" y="43.18" size="1.778" layer="95"/>
 </segment>
-</net>
+<segment>
+<pinref part="C3" gate="G$1" pin="2"/>
+<wire x1="-99.06" y1="88.9" x2="-99.06" y2="81.28" width="0.1524" layer="91"/>
+<wire x1="-99.06" y1="81.28" x2="-99.06" y2="73.66" width="0.1524" layer="91"/>
+<wire x1="-99.06" y1="73.66" x2="-99.06" y2="66.04" width="0.1524" layer="91"/>
+<wire x1="-99.06" y1="66.04" x2="-99.06" y2="58.42" width="0.1524" layer="91"/>
+<wire x1="-99.06" y1="58.42" x2="-106.68" y2="58.42" width="0.1524" layer="91"/>
+<pinref part="C1" gate="G$1" pin="2"/>
+<junction x="-99.06" y="81.28"/>
+<pinref part="C2" gate="G$1" pin="2"/>
+<junction x="-99.06" y="73.66"/>
+<pinref part="C4" gate="G$1" pin="2"/>
+<junction x="-99.06" y="66.04"/>
+<label x="-106.68" y="58.42" size="1.778" layer="95"/>
+</segment>
+</net>
