File: P1001-001 - 16bit CPU/P1001-001-012-320 - Counter ALU/SCH1001-001-012-320 - Counter ALU.brd (EAGLE design)
At the start: 200 x 48 mm, 27 parts, among them IC27 MEGA8535-A, IC51 74LS173D

Commit message: Finished All Boards
Parts:
- added C1, C2, C3, C4: 1uF, rcl:C1206
Connections:
- net GND: now also C1.2, C2.2, C3.2, C4.2
- net VCC: now also C1.1, C2.1, C3.1, C4.1
Routing:
- net VCC: track 402.4 -> 481.9 mm, vias 13 -> 15
- net GND: track 348.6 -> 418.5 mm, vias 13 -> 15
Changed lines of the file:
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@@
 </element>
 <element name="U$1" library="ADAFRUIT" package="4-DIGIT-7-SEGMENT" value="4-DIGIT-7-SEGMENT" x="142" y="2" smashed="yes"/>
+<element name="C3" library="rcl" library_urn="urn:adsk.eagle:library:334" package="C1206" package3d_urn="urn:adsk.eagle:package:23618/2" value="1uF" x="11" y="11" smashed="yes">
+<attribute name="NAME" x="9.73" y="12.27" size="1.27" layer="25"/>
+<attribute name="SPICEPREFIX" value="C" x="11" y="18" size="1.778" layer="27" display="off"/>
+<attribute name="VALUE" x="9.73" y="8.46" size="1.27" layer="27"/>
+</element>
+<element name="C1" library="rcl" library_urn="urn:adsk.eagle:library:334" package="C1206" package3d_urn="urn:adsk.eagle:package:23618/2" value="1uF" x="11" y="38" smashed="yes">
+<attribute name="NAME" x="9.73" y="39.27" size="1.27" layer="25"/>
+<attribute name="SPICEPREFIX" value="C" x="11" y="31" size="1.778" layer="27" display="off"/>
+<attribute name="VALUE" x="9.73" y="35.46" size="1.27" layer="27"/>
+</element>
+<element name="C2" library="rcl" library_urn="urn:adsk.eagle:library:334" package="C1206" package3d_urn="urn:adsk.eagle:package:23618/2" value="1uF" x="196" y="37" smashed="yes" rot="R90">
+<attribute name="NAME" x="194.73" y="35.73" size="1.27" layer="25" rot="R90"/>
+<attribute name="SPICEPREFIX" value="C" x="210" y="32" size="1.778" layer="27" rot="R90" display="off"/>
+<attribute name="VALUE" x="198.54" y="35.73" size="1.27" layer="27" rot="R90"/>
+</element>
+<element name="C4" library="rcl" library_urn="urn:adsk.eagle:library:334" package="C1206" package3d_urn="urn:adsk.eagle:package:23618/2" value="1uF" x="196" y="13" smashed="yes" rot="R90">
+<attribute name="NAME" x="194.73" y="11.73" size="1.27" layer="25" rot="R90"/>
+<attribute name="SPICEPREFIX" value="C" x="210" y="8" size="1.778" layer="27" rot="R90" display="off"/>
+<attribute name="VALUE" x="198.54" y="11.73" size="1.27" layer="27" rot="R90"/>
+</element>
 </elements>
 <signals>
@@
 <via x="100.3554" y="20.955" extent="1-16" drill="0.35"/>
 <via x="119.1006" y="18.5928" extent="1-16" drill="0.35"/>
+<contactref element="C3" pad="2"/>
+<contactref element="C1" pad="2"/>
+<contactref element="C2" pad="2"/>
+<contactref element="C4" pad="2"/>
+<wire x1="12.4206" y1="37.9476" x2="12.4206" y2="11.049" width="0.4572" layer="1"/>
+<wire x1="12.4206" y1="11.049" x2="12.4" y2="11" width="0.4572" layer="1"/>
+<wire x1="12.4206" y1="37.9476" x2="12.4" y2="38" width="0.4572" layer="1"/>
+<wire x1="195.9864" y1="18.8976" x2="195.9864" y2="14.4018" width="0.4572" layer="1"/>
+<wire x1="190.2714" y1="24.6126" x2="195.9864" y2="18.8976" width="0.4572" layer="1"/>
+<wire x1="195.9864" y1="14.4018" x2="196" y2="14.4" width="0.4572" layer="1"/>
+<wire x1="195.9864" y1="37.8714" x2="195.9864" y2="38.3286" width="0.4572" layer="1"/>
+<wire x1="192.1764" y1="34.0614" x2="195.9864" y2="37.8714" width="0.4572" layer="1"/>
+<wire x1="192.1764" y1="27.7368" x2="192.1764" y2="34.0614" width="0.4572" layer="1"/>
+<wire x1="191.5668" y1="27.1272" x2="192.1764" y2="27.7368" width="0.4572" layer="1"/>
+<wire x1="195.9864" y1="38.3286" x2="196" y2="38.4" width="0.4572" layer="1"/>
+<wire x1="191.5668" y1="27.1272" x2="191.445" y2="26.9266" width="0.4572" layer="1"/>
+<wire x1="17.6784" y1="11.049" x2="12.6492" y2="11.049" width="0.4572" layer="1"/>
+<wire x1="21.1836" y1="7.5438" x2="17.6784" y2="11.049" width="0.4572" layer="16"/>
+<wire x1="25.527" y1="7.5438" x2="21.1836" y2="7.5438" width="0.4572" layer="16"/>
+<wire x1="25.8318" y1="7.5438" x2="25.527" y2="7.5438" width="0.4572" layer="1"/>
+<wire x1="26.9748" y1="6.4008" x2="25.8318" y2="7.5438" width="0.4572" layer="1"/>
+<wire x1="12.6492" y1="11.049" x2="12.4" y2="11" width="0.4572" layer="1"/>
+<wire x1="26.9748" y1="6.4008" x2="26.81" y2="5.9266" width="0.4572" layer="1"/>
+<via x="17.6784" y="11.049" extent="1-16" drill="0.35"/>
+<via x="25.527" y="7.5438" extent="1-16" drill="0.35"/>
 </signal>
 <signal name="VCC" class="1">
@@
 <wire x1="19.2024" y1="5.8674" x2="19.19" y2="5.9266" width="0.4572" layer="1"/>
 <wire x1="22.9362" y1="5.8674" x2="23" y2="5.9266" width="0.4572" layer="1"/>
-<wire x1="19.2024" y1="6.096" x2="19.2024" y2="10.5156" width="0.4572" layer="1"/>
+<wire x1="19.2024" y1="6.096" x2="19.2024" y2="9.6774" width="0.4572" layer="1"/>
+<wire x1="19.2024" y1="9.6774" x2="19.2024" y2="10.5156" width="0.4572" layer="1"/>
 <wire x1="19.2024" y1="10.5156" x2="19.2024" y2="12.0396" width="0.4572" layer="1"/>
 <wire x1="19.2024" y1="12.0396" x2="19.19" y2="12.0734" width="0.4572" layer="1"/>
@@
 <wire x1="47.5488" y1="43.053" x2="47.555" y2="43.0734" width="0.4572" layer="1"/>
 <wire x1="26.2128" y1="37.8714" x2="26.175" y2="36.9266" width="0.4572" layer="1"/>
-<wire x1="20.193" y1="41.4528" x2="20.193" y2="10.5156" width="0.4572" layer="16"/>
+<wire x1="20.193" y1="41.4528" x2="20.193" y2="38.0238" width="0.4572" layer="16"/>
+<wire x1="20.193" y1="38.0238" x2="20.193" y2="10.5156" width="0.4572" layer="16"/>
 <wire x1="72.009" y1="22.7838" x2="72.009" y2="20.955" width="0.4572" layer="1"/>
 <wire x1="74.5236" y1="25.2984" x2="72.009" y2="22.7838" width="0.4572" layer="1"/>
@@
 <wire x1="166.116" y1="33.0708" x2="166.19" y2="33.0734" width="0.4572" layer="1"/>
 <wire x1="179.07" y1="41.9862" x2="181.1274" y2="41.9862" width="0.4572" layer="16"/>
-<wire x1="170.307" y1="33.2232" x2="179.07" y2="41.9862" width="0.4572" layer="16"/>
+<wire x1="170.307" y1="33.2232" x2="172.593" y2="35.5092" width="0.4572" layer="16"/>
+<wire x1="172.593" y1="35.5092" x2="179.07" y2="41.9862" width="0.4572" layer="16"/>
 <wire x1="155.829" y1="33.2232" x2="170.307" y2="33.2232" width="0.4572" layer="16"/>
 <wire x1="181.1274" y1="41.9862" x2="181.19" y2="42" width="0.4572" layer="16"/>
@@
 <via x="145.4658" y="33.0708" extent="1-16" drill="0.35"/>
 <via x="155.6766" y="33.0708" extent="1-16" drill="0.35"/>
+<contactref element="C4" pad="1"/>
+<contactref element="C3" pad="1"/>
+<contactref element="C1" pad="1"/>
+<contactref element="C2" pad="1"/>
+<wire x1="196.0626" y1="12.192" x2="196.0626" y2="11.6586" width="0.4572" layer="1"/>
+<wire x1="197.2818" y1="13.4112" x2="196.0626" y2="12.192" width="0.4572" layer="1"/>
+<wire x1="197.2818" y1="34.3662" x2="197.2818" y2="13.4112" width="0.4572" layer="1"/>
+<wire x1="196.0626" y1="35.5854" x2="197.2818" y2="34.3662" width="0.4572" layer="1"/>
+<wire x1="196.0626" y1="11.6586" x2="196" y2="11.6" width="0.4572" layer="1"/>
+<wire x1="196.0626" y1="35.5854" x2="196" y2="35.6" width="0.4572" layer="1"/>
+<wire x1="10.1346" y1="10.9728" x2="9.6012" y2="10.9728" width="0.4572" layer="1"/>
+<wire x1="11.43" y1="9.6774" x2="10.1346" y2="10.9728" width="0.4572" layer="1"/>
+<wire x1="19.2024" y1="9.6774" x2="11.43" y2="9.6774" width="0.4572" layer="1"/>
+<wire x1="9.6012" y1="10.9728" x2="9.6" y2="11" width="0.4572" layer="1"/>
+<wire x1="11.049" y1="38.0238" x2="9.6012" y2="38.0238" width="0.4572" layer="1"/>
+<wire x1="20.193" y1="38.0238" x2="11.049" y2="38.0238" width="0.4572" layer="16"/>
+<wire x1="9.6012" y1="38.0238" x2="9.6" y2="38" width="0.4572" layer="1"/>
+<wire x1="195.7578" y1="12.3444" x2="195.9102" y2="12.3444" width="0.4572" layer="1"/>
+<wire x1="182.7276" y1="25.3746" x2="195.7578" y2="12.3444" width="0.4572" layer="1"/>
+<wire x1="172.593" y1="35.5092" x2="182.7276" y2="25.3746" width="0.4572" layer="16"/>
+<wire x1="195.9102" y1="12.3444" x2="196" y2="11.6" width="0.4572" layer="1"/>
+<via x="11.049" y="38.0238" extent="1-16" drill="0.35"/>
+<via x="182.7276" y="25.3746" extent="1-16" drill="0.35"/>
 </signal>
 <signal name="CLK">
