File: P1001-001 - 16bit CPU/P1001-001-012-320 - Counter ALU/SCH1001-001-012-320 - Counter ALU.sch (EAGLE design)
At the start: 27 parts, among them IC27 MEGA8535-A, IC51 74LS173D

Commit message: Finished All Boards
Parts:
- added C1, C2, C3, C4: 1uF, rcl:C-USC1206
Connections:
- net GND: now also C1.2, C2.2, C3.2, C4.2
- net VCC: now also C1.1, C2.1, C3.1, C4.1
Changed lines of the file:
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@@
 <part name="RN2" library="resistor-dil" library_urn="urn:adsk.eagle:library:342" deviceset="10R-N" device="SOMC" package3d_urn="urn:adsk.eagle:package:24917/1"/>
 <part name="U$1" library="ADAFRUIT" deviceset="4-DIGIT-7-SEGMENT" device=""/>
+<part name="C3" library="rcl" library_urn="urn:adsk.eagle:library:334" deviceset="C-US" device="C1206" package3d_urn="urn:adsk.eagle:package:23618/2" value="1uF"/>
+<part name="C1" library="rcl" library_urn="urn:adsk.eagle:library:334" deviceset="C-US" device="C1206" package3d_urn="urn:adsk.eagle:package:23618/2" value="1uF"/>
+<part name="C2" library="rcl" library_urn="urn:adsk.eagle:library:334" deviceset="C-US" device="C1206" package3d_urn="urn:adsk.eagle:package:23618/2" value="1uF"/>
+<part name="C4" library="rcl" library_urn="urn:adsk.eagle:library:334" deviceset="C-US" device="C1206" package3d_urn="urn:adsk.eagle:package:23618/2" value="1uF"/>
 </parts>
 <sheets>
@@
 <attribute name="VALUE" x="125.095" y="64.008" size="1.778" layer="96" rot="R90"/>
 </instance>
+<instance part="C3" gate="G$1" x="30.48" y="96.52" smashed="yes" rot="R270">
+<attribute name="NAME" x="31.115" y="95.504" size="1.778" layer="95" rot="R270"/>
+<attribute name="VALUE" x="26.289" y="95.504" size="1.778" layer="96" rot="R270"/>
+</instance>
+<instance part="C1" gate="G$1" x="30.48" y="88.9" smashed="yes" rot="R270">
+<attribute name="NAME" x="31.115" y="87.884" size="1.778" layer="95" rot="R270"/>
+<attribute name="VALUE" x="26.289" y="87.884" size="1.778" layer="96" rot="R270"/>
+</instance>
+<instance part="C2" gate="G$1" x="30.48" y="81.28" smashed="yes" rot="R270">
+<attribute name="NAME" x="31.115" y="80.264" size="1.778" layer="95" rot="R270"/>
+<attribute name="VALUE" x="26.289" y="80.264" size="1.778" layer="96" rot="R270"/>
+</instance>
+<instance part="C4" gate="G$1" x="30.48" y="73.66" smashed="yes" rot="R270">
+<attribute name="NAME" x="31.115" y="72.644" size="1.778" layer="95" rot="R270"/>
+<attribute name="VALUE" x="26.289" y="72.644" size="1.778" layer="96" rot="R270"/>
+</instance>
 </instances>
 <busses>
@@
 <wire x1="99.06" y1="124.46" x2="124.46" y2="124.46" width="0.1524" layer="91"/>
 <label x="101.6" y="124.46" size="1.778" layer="95"/>
+</segment>
+<segment>
+<pinref part="C4" gate="G$1" pin="1"/>
+<wire x1="33.02" y1="73.66" x2="33.02" y2="81.28" width="0.1524" layer="91"/>
+<wire x1="33.02" y1="81.28" x2="33.02" y2="88.9" width="0.1524" layer="91"/>
+<wire x1="33.02" y1="88.9" x2="33.02" y2="96.52" width="0.1524" layer="91"/>
+<wire x1="33.02" y1="96.52" x2="33.02" y2="101.6" width="0.1524" layer="91"/>
+<wire x1="33.02" y1="101.6" x2="45.72" y2="101.6" width="0.1524" layer="91"/>
+<pinref part="C3" gate="G$1" pin="1"/>
+<junction x="33.02" y="96.52"/>
+<pinref part="C1" gate="G$1" pin="1"/>
+<junction x="33.02" y="88.9"/>
+<pinref part="C2" gate="G$1" pin="1"/>
+<junction x="33.02" y="81.28"/>
+<label x="38.1" y="101.6" size="1.778" layer="95"/>
 </segment>
 </net>
@@
 <label x="106.68" y="43.18" size="1.778" layer="95"/>
 </segment>
-</net>
+<segment>
+<pinref part="C3" gate="G$1" pin="2"/>
+<wire x1="25.4" y1="96.52" x2="25.4" y2="88.9" width="0.1524" layer="91"/>
+<wire x1="25.4" y1="88.9" x2="25.4" y2="81.28" width="0.1524" layer="91"/>
+<wire x1="25.4" y1="81.28" x2="25.4" y2="73.66" width="0.1524" layer="91"/>
+<wire x1="25.4" y1="73.66" x2="25.4" y2="66.04" width="0.1524" layer="91"/>
+<wire x1="25.4" y1="66.04" x2="17.78" y2="66.04" width="0.1524" layer="91"/>
+<pinref part="C1" gate="G$1" pin="2"/>
+<junction x="25.4" y="88.9"/>
+<pinref part="C2" gate="G$1" pin="2"/>
+<junction x="25.4" y="81.28"/>
+<pinref part="C4" gate="G$1" pin="2"/>
+<junction x="25.4" y="73.66"/>
+<label x="17.78" y="66.04" size="1.778" layer="95"/>
+</segment>
+</net>
