File: P1001-001 - 16bit CPU/P1001-001-006-320 - Program Flash/SCH1001-001-006-320 - Program Flash.sch (EAGLE design)
At the start: 8 parts

Commit message: Add the prototype stuff
Changed lines of the file:
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@@
 <pinref part="MID" gate="B" pin="1"/>
 <wire x1="129.54" y1="45.72" x2="149.86" y2="45.72" width="0.1524" layer="91"/>
+<label x="132.08" y="45.72" size="1.778" layer="95"/>
 </segment>
 </net>
