File: P1001-001 - 16bit CPU/P1001-001-011-320 - RAM/P1001-001-011-320 - RAM.sch (EAGLE design)
At the start: 42 parts, among them IC1 74ALS21D, IC10 74ALS08D, IC2 74283D, IC27 MEGA8535-A, IC3 74ALS04D, IC4 74ALS02D, IC5 74LS32D, IC6 74283D, IC7 74283D, IC8 74283D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

Commit message: Finished All Boards
Parts:
- added C1, C2, C3, C4: 1uF, rcl:C-USC1206
Connections:
- net GND: now also C1.2, C2.2, C3.2, C4.2
- net VCC: now also C1.1, C2.1, C3.1, C4.1

Commit message: Add the prototype stuff
Connections:
- removed net LOWADDR1: IC2A.S1, LOW.9, MEM_LOW.A0
- removed net LOWADDR10: HIGH.5, IC7A.S2, MEM_LOW.A9
- removed net LOWADDR11: IC7A.S3, MEM_LOW.A10, MID.3
- removed net LOWADDR12: HIGH.7, IC7A.S4, MEM_LOW.A11
- removed net LOWADDR13: IC8A.S1, MEM_LOW.A12, MID.5
- removed net LOWADDR14: HIGH.9, IC8A.S2, MEM_LOW.A13
- removed net LOWADDR15: IC8A.S3, MEM_LOW.A14, MID.7
- removed net LOWADDR2: IC2A.S2, MEM_LOW.A1, MID.13
- removed net LOWADDR3: IC2A.S3, LOW.11, MEM_LOW.A2
- removed net LOWADDR4: IC2A.S4, MEM_LOW.A3, MID.15
- removed net LOWADDR5: IC6A.S1, LOW.13, MEM_LOW.A4
- removed net LOWADDR6: HIGH.1, IC6A.S2, MEM_LOW.A5
- removed net LOWADDR7: IC6A.S3, LOW.15, MEM_LOW.A6
- removed net LOWADDR8: HIGH.3, IC6A.S4, MEM_LOW.A7
- removed net LOWADDR9: IC7A.S1, MEM_LOW.A8, MID.1
- new net HIGHADDR1: IC2A.S1, LOW.9, MEM_HIGH.A0
- new net HIGHADDR10: HIGH.5, IC7A.S2, MEM_HIGH.A9
- new net HIGHADDR11: IC7A.S3, MEM_HIGH.A10, MID.3
- new net HIGHADDR12: HIGH.7, IC7A.S4, MEM_HIGH.A11
- new net HIGHADDR13: IC8A.S1, MEM_HIGH.A12, MID.5
- new net HIGHADDR14: HIGH.9, IC8A.S2, MEM_HIGH.A13
- new net HIGHADDR15: IC8A.S3, MEM_HIGH.A14, MID.7
- new net HIGHADDR2: IC2A.S2, MEM_HIGH.A1, MID.13
- new net HIGHADDR3: IC2A.S3, LOW.11, MEM_HIGH.A2
- new net HIGHADDR4: IC2A.S4, MEM_HIGH.A3, MID.15
- new net HIGHADDR5: IC6A.S1, LOW.13, MEM_HIGH.A4
- new net HIGHADDR6: HIGH.1, IC6A.S2, MEM_HIGH.A5
- new net HIGHADDR7: IC6A.S3, LOW.15, MEM_HIGH.A6
- new net HIGHADDR8: HIGH.3, IC6A.S4, MEM_HIGH.A7
- new net HIGHADDR9: IC7A.S1, MEM_HIGH.A8, MID.1
- net ADDR1: now also MEM_LOW.A0; no longer MEM_HIGH.A0
- net ADDR10: now also MEM_LOW.A9; no longer MEM_HIGH.A9
- net ADDR11: now also MEM_LOW.A10; no longer MEM_HIGH.A10
- net ADDR12: now also MEM_LOW.A11; no longer MEM_HIGH.A11
- net ADDR13: now also MEM_LOW.A12; no longer MEM_HIGH.A12
- net ADDR14: now also MEM_LOW.A13; no longer MEM_HIGH.A13
- net ADDR15: now also MEM_LOW.A14; no longer MEM_HIGH.A14
- net ADDR2: now also MEM_LOW.A1; no longer MEM_HIGH.A1
- net ADDR3: now also MEM_LOW.A2; no longer MEM_HIGH.A2
- net ADDR4: now also MEM_LOW.A3; no longer MEM_HIGH.A3
- net ADDR5: now also MEM_LOW.A4; no longer MEM_HIGH.A4
- net ADDR6: now also MEM_LOW.A5; no longer MEM_HIGH.A5
- net ADDR7: now also MEM_LOW.A6; no longer MEM_HIGH.A6
- net ADDR8: now also MEM_LOW.A7; no longer MEM_HIGH.A7
- net ADDR9: now also MEM_LOW.A8; no longer MEM_HIGH.A8
- net ODD_ADDR: now also IC27.(SS)PB4
